Commit message: Add Archer dashboard, perception pipeline, simulation updates, and robot assets

File: ros2_ws/src/archer_description/urdf/archer.urdf.xacro (robot description, xacro)
@@ -2,15 +2,19 @@
 <robot xmlns:xacro="http://www.ros.org/wiki/xacro" name="archer">
   <!-- ========================================================================= -->
-  <!-- Archer: Full Humanoid with Arms & Hands                                 -->
+  <!-- Archer: Overhauled with Professional 1X Technologies Humanoid Meshes      -->
   <!-- ========================================================================= -->
   <xacro:include filename="materials.xacro" />
   <xacro:include filename="inertials.xacro" />
   <xacro:include filename="archer_gazebo.xacro" />
+  <xacro:include filename="archer_control.xacro" />
+  <!-- Unified mesh orientation (aligned with local coordinate frames for both Gazebo and RViz) -->
+  <xacro:property name="mesh_rpy" value="1.5707963 0 1.5707963"/>
+  <!-- Base Link / Frictionless Sled -->
   <link name="base_link">
-    <!-- Invisible Sled for Absolute Stability -->
+    <!-- Invisible Sled for Absolute upright stability -->
     <visual>
       <origin xyz="0 0 0.01" rpy="0 0 0"/>
       <geometry><box size="0.6 0.6 0.01"/></geometry>
-      <material name="transparent"><color rgba="0 0 0 0"/></material>
+      <material name="transparent"/>
     </visual>
     <collision>
@@ -18,136 +22,222 @@
       <geometry><box size="0.6 0.6 0.01"/></geometry>
     </collision>
-    <xacro:box_inertia m="0.1" w="0.6" h="0.6" d="0.01"/>
+    <xacro:box_inertia m="5.0" w="0.6" h="0.6" d="0.01"/>
   </link>
   <joint name="base_joint" type="fixed">
     <parent link="base_link"/><child link="Pelvis"/>
-    <origin xyz="0 0 0.94" rpy="0 0 0"/>
+    <origin xyz="0 0 0.95" rpy="0 0 0"/>
   </joint>
   <gazebo reference="base_link">
-    <!-- Frictionless sled so it doesn't drag -->
+    <!-- Frictionless sled to ensure smooth sliding -->
     <mu1>0.0</mu1><mu2>0.0</mu2>
   </gazebo>
   <!-- Pelvis -->
   <link name="Pelvis">
-    <visual><geometry><box size="0.2 0.3 0.15"/></geometry><material name="blue"/></visual>
+    <!-- Professional 1X Torso Mannequin Mesh -->
+    <visual>
+      <origin xyz="0 0 0" rpy="${mesh_rpy}"/>
+      <geometry>
+        <mesh filename="package://archer_description/meshes/torso.obj" scale="1.0 1.0 1.0"/>
+      </geometry>
+    </visual>
     <collision><geometry><box size="0.2 0.3 0.15"/></geometry></collision>
     <xacro:ballast_inertia m="50.0" w="0.2" h="0.3" d="0.15"/>
   </link>
-  <gazebo reference="Pelvis"><material>Gazebo/Blue</material></gazebo>
-  <!-- Wheels attached to Lower Legs -->
+  <!-- Wheels (Hidden visually inside/under the signature Neo white sneakers) -->
   <link name="left_wheel">
-    <visual><geometry><sphere radius="0.05"/></geometry><material name="black"/></visual>
+    <visual>
+      <origin xyz="0 0 0" rpy="0 0 0"/>
+      <geometry><sphere radius="0.05"/></geometry>
+      <material name="neo_matte_black"/>
+    </visual>
     <collision><geometry><sphere radius="0.05"/></geometry></collision>
     <xacro:sphere_inertia m="2.0" r="0.05"/>
   </link>
   <joint name="left_wheel_joint" type="continuous">
-    <parent link="LeftLowerLeg"/><child link="left_wheel"/>
-    <origin xyz="0 0 -0.4" rpy="0 0 0"/><axis xyz="0 1 0"/>
+    <parent link="base_link"/><child link="left_wheel"/>
+    <origin xyz="0 0.1 0.05" rpy="0 0 0"/><axis xyz="0 1 0"/>
   </joint>
   <link name="right_wheel">
-    <visual><geometry><sphere radius="0.05"/></geometry><material name="black"/></visual>
+    <visual>
+      <origin xyz="0 0 0" rpy="0 0 0"/>
+      <geometry><sphere radius="0.05"/></geometry>
+      <material name="neo_matte_black"/>
+    </visual>
     <collision><geometry><sphere radius="0.05"/></geometry></collision>
     <xacro:sphere_inertia m="2.0" r="0.05"/>
   </link>
   <joint name="right_wheel_joint" type="continuous">
-    <parent link="RightLowerLeg"/><child link="right_wheel"/>
-    <origin xyz="0 0 -0.4" rpy="0 0 0"/><axis xyz="0 1 0"/>
-  </joint>
-  <!-- Trunk -->
+    <parent link="base_link"/><child link="right_wheel"/>
+    <origin xyz="0 -0.1 0.05" rpy="0 0 0"/><axis xyz="0 1 0"/>
+  </joint>
+  <!-- Torso Segment 1: Lower Trunk (Flexible Waist) -->
   <link name="LowerTrunk">
-    <visual><geometry><box size="0.15 0.25 0.2"/></geometry><material name="white"/></visual>
+    <!-- Professional 1X Abdomen Mesh -->
+    <visual>
+      <origin xyz="0 0 0" rpy="${mesh_rpy}"/>
+      <geometry>
+        <mesh filename="package://archer_description/meshes/abdomen.obj" scale="1.0 1.0 1.0"/>
+      </geometry>
+    </visual>
     <collision><geometry><box size="0.15 0.25 0.2"/></geometry></collision>
     <xacro:box_inertia m="5.0" w="0.15" h="0.25" d="0.2"/>
   </link>
-  <joint name="jL5S1_roty" type="fixed">
+  <joint name="jL5S1_roty" type="revolute">
     <parent link="Pelvis"/><child link="LowerTrunk"/><axis xyz="0 1 0"/>
-    <origin xyz="0 0 0.1"/><limit effort="100" velocity="1.0" lower="-0.5" upper="1.5"/>
-  </joint>
-  <gazebo reference="LowerTrunk"><material>Gazebo/White</material></gazebo>
+    <origin xyz="0 0 0.1"/>
+    <limit effort="100" velocity="1.0" lower="-0.5" upper="1.5"/>
+    <dynamics damping="1.5" friction="1.0"/>
+  </joint>
+  <!-- Torso Segment 2: Upper Trunk (Chest / Shoulders) -->
   <link name="UpperTrunk">
-    <visual><geometry><box size="0.15 0.25 0.2"/></geometry><material name="white"/></visual>
+    <!-- Professional 1X Scapula / Shoulder Connector Mesh -->
+    <visual>
+      <origin xyz="0 0 0.1" rpy="${mesh_rpy}"/>
+      <geometry>
+        <mesh filename="package://archer_description/meshes/scapula.obj" scale="1.0 1.0 1.0"/>
+      </geometry>
+    </visual>
     <collision><geometry><box size="0.15 0.25 0.2"/></geometry></collision>
     <xacro:box_inertia m="5.0" w="0.15" h="0.25" d="0.2"/>
   </link>
-  <joint name="jT9T8_roty" type="fixed">
+  <joint name="jT9T8_roty" type="revolute">
     <parent link="LowerTrunk"/><child link="UpperTrunk"/><axis xyz="0 1 0"/>
-    <origin xyz="0 0 0.2"/><limit effort="100" velocity="1.0" lower="-0.2" upper="0.7"/>
-  </joint>
-  <gazebo reference="UpperTrunk"><material>Gazebo/White</material></gazebo>
-  <!-- Head -->
+    <origin xyz="0 0 0.2"/>
+    <limit effort="100" velocity="1.0" lower="-0.2" upper="0.7"/>
+    <dynamics damping="1.5" friction="1.0"/>
+  </joint>
+  <!-- Head (Sleek Visor Helmet with Emotive Rings) -->
   <link name="Head">
-    <visual>
-      <geometry><sphere radius="0.1"/></geometry>
-      <material name="grey"/>
-    </visual>
-    <!-- Left Eye -->
-    <visual>
-      <origin xyz="0.08 0.04 0.05" rpy="0 0 0"/>
-      <geometry><sphere radius="0.02"/></geometry>
-      <material name="black"/>
-    </visual>
-    <!-- Right Eye -->
-    <visual>
-      <origin xyz="0.08 -0.04 0.05" rpy="0 0 0"/>
-      <geometry><sphere radius="0.02"/></geometry>
-      <material name="black"/>
+    <!-- Professional 1X Head Mesh -->
+    <visual>
+      <origin xyz="0 0 0" rpy="${mesh_rpy}"/>
+      <geometry>
+        <mesh filename="package://archer_description/meshes/head.obj" scale="1.0 1.0 1.0"/>
+      </geometry>
     </visual>
     <collision><geometry><sphere radius="0.1"/></geometry></collision>
     <xacro:sphere_inertia m="2.0" r="0.1"/>
   </link>
-  <joint name="jT1C7_roty" type="fixed">
+  <joint name="jT1C7_roty" type="revolute">
     <parent link="UpperTrunk"/><child link="Head"/><axis xyz="0 1 0"/>
-    <origin xyz="0 0 0.2"/><limit effort="10" velocity="1.0" lower="-0.5" upper="0.5"/>
-  </joint>
-  <gazebo reference="Head"><material>Gazebo/Grey</material></gazebo>
-  <!-- LEGS -->
+    <origin xyz="0 0 0.2"/>
+    <limit effort="10" velocity="1.0" lower="-0.5" upper="0.5"/>
+    <dynamics damping="1.5" friction="1.0"/>
+  </joint>
+  <!-- LEGS MACRO (Fully Functional Revolute Thighs, Calves, & Hidden Wheels in Sneakers) -->
   <xacro:macro name="archer_leg" params="side reflect">
     <link name="${side}UpperLeg">
-      <visual><geometry><cylinder radius="0.05" length="0.4"/></geometry><material name="blue"/></visual>
+      <!-- Professional 1X Thigh Mesh -->
+      <visual>
+        <origin xyz="0 0 0" rpy="${mesh_rpy}"/>
+        <geometry>
+          <mesh filename="package://archer_description/meshes/thigh.obj" scale="1.0 1.0 1.0"/>
+        </geometry>
+      </visual>
       <collision><geometry><cylinder radius="0.05" length="0.4"/></geometry></collision>
       <xacro:cylinder_inertia m="3.0" r="0.05" l="0.4"/>
     </link>
-    <joint name="j${side}Hip_roty" type="fixed">
+    <joint name="j${side}Hip_roty" type="revolute">
       <parent link="Pelvis"/><child link="${side}UpperLeg"/><axis xyz="0 1 0"/>
-      <origin xyz="0 ${reflect*0.1} -0.1"/><limit effort="50" velocity="1.0" lower="-1.5" upper="0.5"/>
-    </joint>
-    <gazebo reference="${side}UpperLeg"><material>Gazebo/Blue</material></gazebo>
+      <origin xyz="0 ${reflect*0.1} -0.1"/>
+      <limit effort="50" velocity="1.0" lower="-1.5" upper="0.5"/>
+      <dynamics damping="1.5" friction="1.0"/>
+    </joint>
     <link name="${side}LowerLeg">
-      <visual><geometry><cylinder radius="0.04" length="0.4"/></geometry><material name="blue"/></visual>
+      <!-- Professional 1X Shin Mesh -->
+      <visual>
+        <origin xyz="0 0 0" rpy="${mesh_rpy}"/>
+        <geometry>
+          <mesh filename="package://archer_description/meshes/shin.obj" scale="1.0 1.0 1.0"/>
+        </geometry>
+      </visual>
+      <!-- signature 1X NEO Athletic Knit Sneaker at bottom -->
+      <!-- White sole -->
+      <visual>
+        <origin xyz="0.04 0 -0.34" rpy="0 0 0"/>
+        <geometry><box size="0.22 0.10 0.04"/></geometry>
+        <material name="neo_sneaker_white"/>
+      </visual>
+      <!-- Black sole tread -->
+      <visual>
+        <origin xyz="0.04 0 -0.36" rpy="0 0 0"/>
+        <geometry><box size="0.224 0.104 0.01"/></geometry>
+        <material name="neo_matte_black"/>
+      </visual>
+      <!-- Knit sneaker upper body (Knit grey) -->
+      <visual>
+        <origin xyz="0.03 0 -0.28" rpy="0 0.15 0"/>
+        <geometry><box size="0.18 0.09 0.08"/></geometry>
+        <material name="neo_knit_gray"/>
+      </visual>
+      <!-- Sneaker heel cap wrap (Matte black) -->
+      <visual>
+        <origin xyz="-0.04 0 -0.29" rpy="0 0 0"/>
+        <geometry><box size="0.05 0.092 0.082"/></geometry>
+        <material name="neo_matte_black"/>
+      </visual>
+      <!-- White sneaker collar / ankle cuff -->
+      <visual>
+        <origin xyz="0 0 -0.22" rpy="0 0 0"/>
+        <geometry><cylinder radius="0.045" length="0.04"/></geometry>
+        <material name="neo_sneaker_white"/>
+      </visual>
       <collision><geometry><cylinder radius="0.04" length="0.4"/></geometry></collision>
       <xacro:cylinder_inertia m="2.0" r="0.04" l="0.4"/>
     </link>
-    <joint name="j${side}Knee_roty" type="fixed">
+    <joint name="j${side}Knee_roty" type="revolute">
       <parent link="${side}UpperLeg"/><child link="${side}LowerLeg"/><axis xyz="0 1 0"/>
-      <origin xyz="0 0 -0.4"/><limit effort="50" velocity="1.0" lower="0" upper="2.0"/>
-    </joint>
-    <gazebo reference="${side}LowerLeg"><material>Gazebo/Blue</material></gazebo>
+      <origin xyz="0 0 -0.4"/>
+      <limit effort="50" velocity="1.0" lower="0" upper="2.0"/>
+      <dynamics damping="1.5" friction="1.0"/>
+    </joint>
   </xacro:macro>
   <xacro:archer_leg side="Left" reflect="1"/>
   <xacro:archer_leg side="Right" reflect="-1"/>
-  <!-- ARMS -->
+  <!-- ARMS MACRO (Fully Functional Revolute Shoulders & Elbows, with Mitten Hands) -->
   <xacro:macro name="archer_arm" params="side reflect">
     <link name="${side}UpperArm">
-      <visual><geometry><cylinder radius="0.03" length="0.3"/></geometry><material name="white"/></visual>
+      <!-- Professional 1X Upper Arm Mesh -->
+      <visual>
+        <origin xyz="0 0 0" rpy="${mesh_rpy}"/>
+        <geometry>
+          <mesh filename="package://archer_description/meshes/upper_arm.obj" scale="1.0 1.0 1.0"/>
+        </geometry>
+      </visual>
       <collision><geometry><cylinder radius="0.03" length="0.3"/></geometry></collision>
       <xacro:cylinder_inertia m="1.5" r="0.03" l="0.3"/>
     </link>
-    <joint name="j${side}Shoulder_roty" type="fixed">
+    <joint name="j${side}Shoulder_roty" type="revolute">
       <parent link="UpperTrunk"/><child link="${side}UpperArm"/><axis xyz="0 1 0"/>
-      <origin xyz="0 ${reflect*0.2} 0.1"/><limit effort="30" velocity="1.0" lower="-1.5" upper="1.5"/>
-    </joint>
-    <gazebo reference="${side}UpperArm"><material>Gazebo/White</material></gazebo>
+      <origin xyz="0 ${reflect*0.2} 0.1"/>
+      <limit effort="30" velocity="1.0" lower="-1.5" upper="1.5"/>
+      <dynamics damping="1.5" friction="1.0"/>
+    </joint>
     <link name="${side}LowerArm">
-      <visual><geometry><cylinder radius="0.02" length="0.3"/></geometry><material name="white"/></visual>
+      <!-- Professional 1X Forearm Mesh -->
+      <visual>
+        <origin xyz="0 0 0" rpy="${mesh_rpy}"/>
+        <geometry>
+          <mesh filename="package://archer_description/meshes/forearm.obj" scale="1.0 1.0 1.0"/>
+        </geometry>
+      </visual>
       <collision><geometry><cylinder radius="0.02" length="0.3"/></geometry></collision>
       <xacro:cylinder_inertia m="1.0" r="0.02" l="0.3"/>
     </link>
-    <joint name="j${side}Elbow_roty" type="fixed">
+    <joint name="j${side}Elbow_roty" type="revolute">
       <parent link="${side}UpperArm"/><child link="${side}LowerArm"/><axis xyz="0 1 0"/>
-      <origin xyz="0 0 -0.3"/><limit effort="30" velocity="1.0" lower="-2.0" upper="0"/>
-    </joint>
-    <gazebo reference="${side}LowerArm"><material>Gazebo/White</material></gazebo>
+      <origin xyz="0 0 -0.3"/>
+      <limit effort="30" velocity="1.0" lower="-2.0" upper="0"/>
+      <dynamics damping="1.5" friction="1.0"/>
+    </joint>
+    <!-- Hand (Robotic Mitten styled in high-fidelity 1X Neo aesthetic) -->
     <link name="${side}Hand">
-      <visual><geometry><sphere radius="0.04"/></geometry><material name="grey"/></visual>
+      <!-- Professional 1X Palm Mesh -->
+      <visual>
+        <origin xyz="0 0 0" rpy="${mesh_rpy}"/>
+        <geometry>
+          <mesh filename="package://archer_description/meshes/palm.obj" scale="1.0 1.0 1.0"/>
+        </geometry>
+      </visual>
       <collision><geometry><sphere radius="0.04"/></geometry></collision>
       <xacro:sphere_inertia m="0.5" r="0.04"/>
@@ -157,5 +247,4 @@
       <origin xyz="0 0 -0.15"/>
     </joint>
-    <gazebo reference="${side}Hand"><material>Gazebo/Grey</material></gazebo>
   </xacro:macro>
   <xacro:archer_arm side="Left" reflect="1"/>

File: ros2_ws/src/archer_description/urdf/archer_control.xacro (robot description, xacro)
@@ -46,4 +46,7 @@
     <plugin filename="libgz_ros2_control-system" name="gz_ros2_control::GazeboSimROS2ControlPlugin">
       <parameters>$(find archer_description)/config/controllers.yaml</parameters>
+      <ros>
+        <namespace>/</namespace>
+      </ros>
     </plugin>
   </gazebo>

File: ros2_ws/src/archer_description/urdf/archer_gazebo.xacro (robot description, xacro)
@@ -13,6 +13,6 @@
       <wheel_separation>0.2</wheel_separation>
       <wheel_radius>0.05</wheel_radius>
-      <max_linear_acceleration>0.5</max_linear_acceleration>
-      <max_angular_acceleration>1.0</max_angular_acceleration>
+      <max_linear_acceleration>1.5</max_linear_acceleration>
+      <max_angular_acceleration>2.5</max_angular_acceleration>
       <max_velocity>2.0</max_velocity>
       <odom_publish_frequency>50</odom_publish_frequency>
@@ -20,4 +20,5 @@
       <odom_topic>/odom</odom_topic>
       <tf_topic>/tf</tf_topic>
+      <publish_odom_tf>true</publish_odom_tf>
       <frame_id>odom</frame_id>
       <child_frame_id>base_link</child_frame_id>
@@ -26,15 +27,78 @@
   <!-- Sensors Definition -->
   <gazebo reference="Head">
+    <!-- RGB Camera (Proven to work on WSL) -->
     <sensor name="head_camera" type="camera">
       <pose>0.2 0 0.1 0 0 0</pose>
       <always_on>1</always_on>
-      <update_rate>30</update_rate>
+      <update_rate>10</update_rate>
       <visualize>true</visualize>
       <topic>/archer/camera/image_raw</topic>
+      <gz_frame_id>Head</gz_frame_id>
+      <frame_id>Head</frame_id>
       <camera>
         <horizontal_fov>1.047</horizontal_fov>
-        <image><width>640</width><height>480</height></image>
+        <image>
+          <width>320</width>
+          <height>240</height>
+          <format>R8G8B8</format>
+        </image>
         <clip><near>0.1</near><far>100</far></clip>
       </camera>
+    </sensor>
+    <!-- Depth Camera for 3D Voxels -->
+    <sensor name="head_camera_depth" type="depth_camera">
+      <pose>0.2 0 0.1 0 0 0</pose>
+      <always_on>1</always_on>
+      <update_rate>5</update_rate>
+      <visualize>false</visualize>
+      <topic>/archer/camera/depth</topic>
+      <gz_frame_id>Head</gz_frame_id>
+      <frame_id>Head</frame_id>
+      <camera>
+        <horizontal_fov>1.047</horizontal_fov>
+        <image>
+          <width>320</width>
+          <height>240</height>
+        </image>
+        <clip><near>0.1</near><far>10.0</far></clip>
+      </camera>
+    </sensor>
+    <!-- Lidar (aligned perfectly with eyes) -->
+    <sensor name="base_lidar" type="gpu_lidar">
+      <pose>0.2 0 0.1 0 0 0</pose>
+      <always_on>true</always_on>
+      <visualize>false</visualize>
+      <update_rate>10</update_rate>
+      <topic>/scan</topic>
+      <gz_frame_id>Head</gz_frame_id>
+      <frame_id>Head</frame_id>
+      <lidar>
+        <scan>
+          <horizontal>
+            <samples>220</samples>
+            <resolution>1</resolution>
+            <min_angle>-1.91986</min_angle>
+            <max_angle>1.91986</max_angle>
+          </horizontal>
+        </scan>
+        <range>
+          <min>0.15</min>
+          <max>12.0</max>
+          <resolution>0.01</resolution>
+        </range>
+      </lidar>
+    </sensor>
+  </gazebo>
+  <!-- IMU for SLAM and Sensor Fusion -->
+  <gazebo reference="base_link">
+    <!-- IMU -->
+    <sensor name="imu_sensor" type="imu">
+      <pose>0 0 0 0 0 0</pose>
+      <always_on>1</always_on>
+      <update_rate>50</update_rate>
+      <visualize>true</visualize>
+      <topic>/imu</topic>
+      <gz_frame_id>base_link</gz_frame_id>
+      <frame_id>base_link</frame_id>
     </sensor>
   </gazebo>

File: ros2_ws/src/archer_description/urdf/archer_sensors.xacro (robot description, xacro)
@@ -9,5 +9,5 @@
       <pose>0 0 0.1 0 0 0</pose>
       <topic>/scan</topic>
-      <visualize>true</visualize>
+      <visualize>false</visualize>
       <update_rate>10</update_rate>
       <lidar>

File: ros2_ws/src/archer_description/urdf/materials.xacro (robot description, xacro)
@@ -1,4 +1,32 @@
 <?xml version="1.0"?>
 <robot xmlns:xacro="http://www.ros.org/wiki/xacro">
+  <!-- ========================================================================= -->
+  <!-- 1X Neo Premium Palette (Domestic Humanoid Design)                          -->
+  <!-- ========================================================================= -->
+  <!-- Premium space-grey knit jumpsuit texture representation -->
+  <material name="neo_knit_gray">
+    <color rgba="0.36 0.36 0.38 1.0"/>
+  </material>
+  <!-- Dark charcoal for underlying joints and compliant rubberized covers -->
+  <material name="neo_matte_black">
+    <color rgba="0.08 0.08 0.09 1.0"/>
+  </material>
+  <!-- Deep glossy black for the head visor faceplate -->
+  <material name="neo_visor_black">
+    <color rgba="0.015 0.015 0.02 1.0"/>
+  </material>
+  <!-- High-contrast pure white for the signature sneakers and chest grilles -->
+  <material name="neo_sneaker_white">
+    <color rgba="0.96 0.96 0.97 1.0"/>
+  </material>
+  <!-- Friendly amber-orange status LED glow for the ears and chest rings -->
+  <material name="neo_led_glow">
+    <color rgba="0.96 0.48 0.08 1.0"/>
+  </material>
+  <!-- Completely transparent helper material -->
+  <material name="transparent">
+    <color rgba="0.0 0.0 0.0 0.0"/>
+  </material>
+  <!-- Basic blue and white kept for compatibility if needed -->
   <material name="blue">
     <color rgba="0.0 0.0 0.8 1.0"/>
@@ -13,6 +41,3 @@
     <color rgba="0.0 0.0 0.0 1.0"/>
   </material>
-  <material name="red">
-    <color rgba="0.8 0.0 0.0 1.0"/>
-  </material>
 </robot>
