Commit message: FInal Fixex, Readme

File: ros2_ws/src/archer_description/urdf/archer.urdf.xacro (robot description, xacro)
@@ -7,28 +7,55 @@
   <xacro:include filename="inertials.xacro" />
   <xacro:include filename="archer_gazebo.xacro" />
-  <xacro:include filename="archer_control.xacro" />
   <!-- Unified mesh orientation (aligned with local coordinate frames for both Gazebo and RViz) -->
   <xacro:property name="mesh_rpy" value="1.5707963 0 1.5707963"/>
-  <!-- Base Link / Frictionless Sled -->
+  <!-- Base Link -->
   <link name="base_link">
-    <!-- Invisible Sled for Absolute upright stability -->
-    <visual>
-      <origin xyz="0 0 0.01" rpy="0 0 0"/>
-      <geometry><box size="0.6 0.6 0.01"/></geometry>
-      <material name="transparent"/>
-    </visual>
+    <!-- Raised collision so it doesn't drag -->
     <collision>
-      <origin xyz="0 0 0.01" rpy="0 0 0"/>
-      <geometry><box size="0.6 0.6 0.01"/></geometry>
+      <origin xyz="0 0 0.15" rpy="0 0 0"/>
+      <geometry><box size="0.6 0.6 0.1"/></geometry>
     </collision>
-    <xacro:box_inertia m="5.0" w="0.6" h="0.6" d="0.01"/>
-  </link>
+    <xacro:box_inertia m="50.0" w="0.6" h="0.6" d="0.1"/>
+  </link>
+  <!-- Caster Wheels for upright stability and traction -->
+  <link name="front_caster">
+    <collision>
+      <origin xyz="0 0 0" rpy="0 0 0"/>
+      <geometry><sphere radius="0.04"/></geometry>
+    </collision>
+    <xacro:sphere_inertia m="1.0" r="0.04"/>
+  </link>
+  <joint name="front_caster_joint" type="fixed">
+    <parent link="base_link"/>
+    <child link="front_caster"/>
+    <origin xyz="0.25 0 0.04" rpy="0 0 0"/>
+  </joint>
+  <link name="rear_caster">
+    <collision>
+      <origin xyz="0 0 0" rpy="0 0 0"/>
+      <geometry><sphere radius="0.04"/></geometry>
+    </collision>
+    <xacro:sphere_inertia m="1.0" r="0.04"/>
+  </link>
+  <joint name="rear_caster_joint" type="fixed">
+    <parent link="base_link"/>
+    <child link="rear_caster"/>
+    <origin xyz="-0.25 0 0.04" rpy="0 0 0"/>
+  </joint>
   <joint name="base_joint" type="fixed">
     <parent link="base_link"/><child link="Pelvis"/>
     <origin xyz="0 0 0.95" rpy="0 0 0"/>
   </joint>
-  <gazebo reference="base_link">
-    <!-- Frictionless sled to ensure smooth sliding -->
+  <gazebo reference="front_caster">
     <mu1>0.0</mu1><mu2>0.0</mu2>
+  </gazebo>
+  <gazebo reference="rear_caster">
+    <mu1>0.0</mu1><mu2>0.0</mu2>
+  </gazebo>
+  <gazebo reference="left_wheel">
+    <mu1>1000.0</mu1><mu2>1000.0</mu2>
+  </gazebo>
+  <gazebo reference="right_wheel">
+    <mu1>1000.0</mu1><mu2>1000.0</mu2>
   </gazebo>
   <!-- Pelvis -->
@@ -42,5 +69,5 @@
     </visual>
     <collision><geometry><box size="0.2 0.3 0.15"/></geometry></collision>
-    <xacro:ballast_inertia m="50.0" w="0.2" h="0.3" d="0.15"/>
+    <xacro:ballast_inertia m="5.0" w="0.2" h="0.3" d="0.15"/>
   </link>
   <!-- Wheels (Hidden visually inside/under the signature Neo white sneakers) -->
@@ -83,9 +110,7 @@
     <xacro:box_inertia m="5.0" w="0.15" h="0.25" d="0.2"/>
   </link>
-  <joint name="jL5S1_roty" type="revolute">
-    <parent link="Pelvis"/><child link="LowerTrunk"/><axis xyz="0 1 0"/>
-    <origin xyz="0 0 0.1"/>
-    <limit effort="100" velocity="1.0" lower="-0.5" upper="1.5"/>
-    <dynamics damping="1.5" friction="1.0"/>
+  <joint name="jL5S1_roty" type="fixed">
+    <parent link="Pelvis"/><child link="LowerTrunk"/>
+    <origin xyz="0 0 0.1" rpy="0 0 0"/>
   </joint>
   <!-- Torso Segment 2: Upper Trunk (Chest / Shoulders) -->
@@ -101,9 +126,7 @@
     <xacro:box_inertia m="5.0" w="0.15" h="0.25" d="0.2"/>
   </link>
-  <joint name="jT9T8_roty" type="revolute">
-    <parent link="LowerTrunk"/><child link="UpperTrunk"/><axis xyz="0 1 0"/>
-    <origin xyz="0 0 0.2"/>
-    <limit effort="100" velocity="1.0" lower="-0.2" upper="0.7"/>
-    <dynamics damping="1.5" friction="1.0"/>
+  <joint name="jT9T8_roty" type="fixed">
+    <parent link="LowerTrunk"/><child link="UpperTrunk"/>
+    <origin xyz="0 0 0.2" rpy="0 0 0"/>
   </joint>
   <!-- Head (Sleek Visor Helmet with Emotive Rings) -->
@@ -119,9 +142,26 @@
     <xacro:sphere_inertia m="2.0" r="0.1"/>
   </link>
-  <joint name="jT1C7_roty" type="revolute">
-    <parent link="UpperTrunk"/><child link="Head"/><axis xyz="0 1 0"/>
-    <origin xyz="0 0 0.2"/>
-    <limit effort="10" velocity="1.0" lower="-0.5" upper="0.5"/>
-    <dynamics damping="1.5" friction="1.0"/>
+  <joint name="jT1C7_roty" type="fixed">
+    <parent link="UpperTrunk"/><child link="Head"/>
+    <origin xyz="0 0 0.3" rpy="0 0 0"/>
+  </joint>
+  <!-- Sensor Links (for perfect Gazebo/ROS TF alignment) -->
+  <link name="head_camera_link"/>
+  <joint name="head_camera_joint" type="fixed">
+    <parent link="Head"/>
+    <child link="head_camera_link"/>
+    <origin xyz="0.2 0 0.1" rpy="0 0 0"/>
+  </joint>
+  <link name="base_lidar_link"/>
+  <joint name="base_lidar_joint" type="fixed">
+    <parent link="Head"/>
+    <child link="base_lidar_link"/>
+    <origin xyz="0.2 0 0.1" rpy="0 0 0"/>
+  </joint>
+  <link name="torso_lidar_link"/>
+  <joint name="torso_lidar_joint" type="fixed">
+    <parent link="Pelvis"/>
+    <child link="torso_lidar_link"/>
+    <origin xyz="0 0 0.20" rpy="0 0 0"/>
   </joint>
   <!-- LEGS MACRO (Fully Functional Revolute Thighs, Calves, & Hidden Wheels in Sneakers) -->
@@ -138,9 +178,7 @@
       <xacro:cylinder_inertia m="3.0" r="0.05" l="0.4"/>
     </link>
-    <joint name="j${side}Hip_roty" type="revolute">
-      <parent link="Pelvis"/><child link="${side}UpperLeg"/><axis xyz="0 1 0"/>
-      <origin xyz="0 ${reflect*0.1} -0.1"/>
-      <limit effort="50" velocity="1.0" lower="-1.5" upper="0.5"/>
-      <dynamics damping="1.5" friction="1.0"/>
+    <joint name="j${side}Hip_roty" type="fixed">
+      <parent link="Pelvis"/><child link="${side}UpperLeg"/>
+      <origin xyz="0 ${reflect*0.1} -0.1" rpy="0 0 0"/>
     </joint>
     <link name="${side}LowerLeg">
@@ -186,9 +224,7 @@
       <xacro:cylinder_inertia m="2.0" r="0.04" l="0.4"/>
     </link>
-    <joint name="j${side}Knee_roty" type="revolute">
-      <parent link="${side}UpperLeg"/><child link="${side}LowerLeg"/><axis xyz="0 1 0"/>
-      <origin xyz="0 0 -0.4"/>
-      <limit effort="50" velocity="1.0" lower="0" upper="2.0"/>
-      <dynamics damping="1.5" friction="1.0"/>
+    <joint name="j${side}Knee_roty" type="fixed">
+      <parent link="${side}UpperLeg"/><child link="${side}LowerLeg"/>
+      <origin xyz="0 0 -0.4" rpy="0 0 0"/>
     </joint>
   </xacro:macro>
@@ -208,9 +244,7 @@
       <xacro:cylinder_inertia m="1.5" r="0.03" l="0.3"/>
     </link>
-    <joint name="j${side}Shoulder_roty" type="revolute">
-      <parent link="UpperTrunk"/><child link="${side}UpperArm"/><axis xyz="0 1 0"/>
-      <origin xyz="0 ${reflect*0.2} 0.1"/>
-      <limit effort="30" velocity="1.0" lower="-1.5" upper="1.5"/>
-      <dynamics damping="1.5" friction="1.0"/>
+    <joint name="j${side}Shoulder_roty" type="fixed">
+      <parent link="UpperTrunk"/><child link="${side}UpperArm"/>
+      <origin xyz="0 ${reflect*0.2} 0.1" rpy="0 0 0"/>
     </joint>
     <link name="${side}LowerArm">
@@ -225,9 +259,7 @@
       <xacro:cylinder_inertia m="1.0" r="0.02" l="0.3"/>
     </link>
-    <joint name="j${side}Elbow_roty" type="revolute">
-      <parent link="${side}UpperArm"/><child link="${side}LowerArm"/><axis xyz="0 1 0"/>
-      <origin xyz="0 0 -0.3"/>
-      <limit effort="30" velocity="1.0" lower="-2.0" upper="0"/>
-      <dynamics damping="1.5" friction="1.0"/>
+    <joint name="j${side}Elbow_roty" type="fixed">
+      <parent link="${side}UpperArm"/><child link="${side}LowerArm"/>
+      <origin xyz="0 0 -0.3" rpy="0 0 0"/>
     </joint>
     <!-- Hand (Robotic Mitten styled in high-fidelity 1X Neo aesthetic) -->
@@ -235,5 +267,5 @@
       <!-- Professional 1X Palm Mesh -->
       <visual>
-        <origin xyz="0 0 0" rpy="${mesh_rpy}"/>
+        <origin xyz="0 0 0" rpy="1.5707963 3.14159265 1.5707963"/>
         <geometry>
           <mesh filename="package://archer_description/meshes/palm.obj" scale="1.0 1.0 1.0"/>

File: ros2_ws/src/archer_description/urdf/archer_control.xacro (robot description, xacro)
@@ -5,41 +5,5 @@
       <plugin>gz_ros2_control/GazeboSimSystem</plugin>
     </hardware>
-    <!-- Torso Joints -->
-    <joint name="jL5S1_roty">
-      <command_interface name="position"><param name="min">-0.5</param><param name="max">1.5</param></command_interface>
-      <state_interface name="position"/><state_interface name="velocity"/>
-    </joint>
-    <joint name="jT9T8_roty">
-      <command_interface name="position"><param name="min">-0.2</param><param name="max">0.7</param></command_interface>
-      <state_interface name="position"/><state_interface name="velocity"/>
-    </joint>
-    <joint name="jT1C7_roty">
-      <command_interface name="position"><param name="min">-0.5</param><param name="max">0.5</param></command_interface>
-      <state_interface name="position"/><state_interface name="velocity"/>
-    </joint>
-    <!-- Leg Joints -->
-    <xacro:macro name="leg_control" params="side">
-      <joint name="j${side}Hip_roty">
-        <command_interface name="position"><param name="min">-1.5</param><param name="max">0.5</param></command_interface>
-        <state_interface name="position"/><state_interface name="velocity"/>
-      </joint>
-      <joint name="j${side}Knee_roty">
-        <command_interface name="position"><param name="min">0</param><param name="max">2.0</param></command_interface>
-        <state_interface name="position"/><state_interface name="velocity"/>
-      </joint>
-    </xacro:macro>
-    <xacro:leg_control side="Left"/><xacro:leg_control side="Right"/>
-    <!-- Arm Joints -->
-    <xacro:macro name="arm_control" params="side">
-      <joint name="j${side}Shoulder_roty">
-        <command_interface name="position"><param name="min">-1.5</param><param name="max">1.5</param></command_interface>
-        <state_interface name="position"/><state_interface name="velocity"/>
-      </joint>
-      <joint name="j${side}Elbow_roty">
-        <command_interface name="position"><param name="min">-2.0</param><param name="max">0</param></command_interface>
-        <state_interface name="position"/><state_interface name="velocity"/>
-      </joint>
-    </xacro:macro>
-    <xacro:arm_control side="Left"/><xacro:arm_control side="Right"/>
+    <!-- No limb or torso joints needed, they are all fixed -->
   </ros2_control>
   <gazebo>

File: ros2_ws/src/archer_description/urdf/archer_gazebo.xacro (robot description, xacro)
@@ -20,5 +20,5 @@
       <odom_topic>/odom</odom_topic>
       <tf_topic>/tf</tf_topic>
-      <publish_odom_tf>false</publish_odom_tf>
+      <publish_odom_tf>true</publish_odom_tf>
       <frame_id>odom</frame_id>
       <child_frame_id>base_link</child_frame_id>
@@ -26,14 +26,14 @@
   </gazebo>
   <!-- Sensors Definition -->
-  <gazebo reference="Head">
+  <gazebo reference="head_camera_link">
     <!-- RGB Camera (Proven to work on WSL) -->
     <sensor name="head_camera" type="camera">
-      <pose>0.2 0 0.1 0 0 0</pose>
+      <pose>0 0 0 0 0 0</pose>
       <always_on>1</always_on>
-      <update_rate>10</update_rate>
+      <update_rate>2</update_rate>
       <visualize>true</visualize>
       <topic>/archer/camera/image_raw</topic>
-      <gz_frame_id>Head</gz_frame_id>
-      <frame_id>Head</frame_id>
+      <gz_frame_id>head_camera_link</gz_frame_id>
+      <frame_id>head_camera_link</frame_id>
       <camera>
         <horizontal_fov>1.047</horizontal_fov>
@@ -48,11 +48,11 @@
     <!-- Depth Camera for 3D Voxels -->
     <sensor name="head_camera_depth" type="depth_camera">
-      <pose>0.2 0 0.1 0 0 0</pose>
+      <pose>0 0 0 0 0 0</pose>
       <always_on>1</always_on>
       <update_rate>5</update_rate>
       <visualize>false</visualize>
       <topic>/archer/camera/depth</topic>
-      <gz_frame_id>Head</gz_frame_id>
-      <frame_id>Head</frame_id>
+      <gz_frame_id>head_camera_link</gz_frame_id>
+      <frame_id>head_camera_link</frame_id>
       <camera>
         <horizontal_fov>1.047</horizontal_fov>
@@ -64,13 +64,16 @@
       </camera>
     </sensor>
+  </gazebo>
+  <gazebo reference="base_lidar_link">
+    <!-- Lidar on Head to ensure horizontal scans -->
     <!-- Lidar (CPU lidar - gpu_lidar silently fails in WSL without hardware GPU) -->
     <sensor name="base_lidar" type="gpu_lidar">
-      <pose>0.2 0 0.1 0 0 0</pose>
+      <pose>0 0 0 0 0 0</pose>
       <always_on>true</always_on>
       <visualize>true</visualize>
       <update_rate>10</update_rate>
       <topic>/scan</topic>
-      <gz_frame_id>Head</gz_frame_id>
-      <frame_id>Head</frame_id>
+      <gz_frame_id>base_lidar_link</gz_frame_id>
+      <frame_id>base_lidar_link</frame_id>
       <lidar>
         <scan>
@@ -83,5 +86,32 @@
         </scan>
         <range>
-          <min>0.45</min>
+          <min>0.40</min>
+          <max>12.0</max>
+          <resolution>0.01</resolution>
+        </range>
+      </lidar>
+    </sensor>
+  </gazebo>
+  <!-- Torso Lidar (360 degrees, ignores body) -->
+  <gazebo reference="torso_lidar_link">
+    <sensor name="torso_lidar" type="gpu_lidar">
+      <pose>0 0 0 0 0 0</pose>
+      <always_on>true</always_on>
+      <visualize>true</visualize>
+      <update_rate>10</update_rate>
+      <topic>/scan_torso</topic>
+      <gz_frame_id>torso_lidar_link</gz_frame_id>
+      <frame_id>torso_lidar_link</frame_id>
+      <lidar>
+        <scan>
+          <horizontal>
+            <samples>360</samples>
+            <resolution>1</resolution>
+            <min_angle>-3.14159</min_angle>
+            <max_angle>3.14159</max_angle>
+          </horizontal>
+        </scan>
+        <range>
+          <min>0.40</min>
           <max>12.0</max>
           <resolution>0.01</resolution>

File: ros2_ws/src/archer_description/urdf/archer_sensors.xacro (robot description, xacro)
@@ -5,7 +5,7 @@
   <!-- ========================================================================= -->
   <!-- LiDAR (GPU Lidar for Harmonic) -->
-  <gazebo reference="Head">
-    <sensor type="gpu_lidar" name="head_lidar">
-      <pose>0 0 0.1 0 0 0</pose>
+  <gazebo reference="Pelvis">
+    <sensor type="gpu_lidar" name="body_lidar">
+      <pose>0 0 0.2 0 0 0</pose>
       <topic>/scan</topic>
       <visualize>false</visualize>

File: ros2_ws/src/archer_description/urdf/inertials.xacro (robot description, xacro)
@@ -34,6 +34,6 @@
   <xacro:macro name="ballast_inertia" params="m w h d">
     <inertial>
-      <!-- Optimized anchor: -0.8m for rock-solid stability without simulation glitches -->
-      <origin xyz="0 0 -0.8" rpy="0 0 0"/>
+      <!-- Standard anchor to avoid physics solver glitches -->
+      <origin xyz="0 0 0" rpy="0 0 0"/>
       <mass value="${m}"/>
       <inertia ixx="100.0" ixy="0.0" ixz="0.0"
