Commit message: feat(system): integrate NVIDIA cuVSLAM stereo VO, tune EKF & Nav2 stack, update bridge & comprehensive README hook

File: ros2_ws/src/archer_description/urdf/archer.urdf.xacro (robot description, xacro)
@@ -1,4 +1,5 @@
 <?xml version="1.0"?>
 <robot xmlns:xacro="http://www.ros.org/wiki/xacro" name="archer">
+  <xacro:arg name="use_cuvslam" default="false"/>
   <!-- ========================================================================= -->
   <!-- Archer: Overhauled with Professional 1X Technologies Humanoid Meshes      -->
@@ -9,4 +10,13 @@
   <!-- Unified mesh orientation (aligned with local coordinate frames for both Gazebo and RViz) -->
   <xacro:property name="mesh_rpy" value="1.5707963 0 1.5707963"/>
+  <!-- Base Footprint (Root Link) -->
+  <link name="base_footprint">
+    <xacro:box_inertia m="5.0" w="0.6" h="0.6" d="0.1"/>
+  </link>
+  <joint name="base_footprint_joint" type="fixed">
+    <parent link="base_footprint"/>
+    <child link="base_link"/>
+    <origin xyz="0 0 0" rpy="0 0 0"/>
+  </joint>
   <!-- Base Link -->
   <link name="base_link">
@@ -16,5 +26,5 @@
       <geometry><box size="0.6 0.6 0.1"/></geometry>
     </collision>
-    <xacro:box_inertia m="50.0" w="0.6" h="0.6" d="0.1"/>
+    <xacro:box_inertia m="5.0" w="0.6" h="0.6" d="0.1"/>
   </link>
   <!-- Caster Wheels for upright stability and traction -->
@@ -26,8 +36,9 @@
     <xacro:sphere_inertia m="1.0" r="0.04"/>
   </link>
-  <joint name="front_caster_joint" type="fixed">
+  <joint name="front_caster_joint" type="continuous">
     <parent link="base_link"/>
     <child link="front_caster"/>
     <origin xyz="0.25 0 0.04" rpy="0 0 0"/>
+    <axis xyz="0 1 0"/>
   </joint>
   <link name="rear_caster">
@@ -38,8 +49,35 @@
     <xacro:sphere_inertia m="1.0" r="0.04"/>
   </link>
-  <joint name="rear_caster_joint" type="fixed">
+  <joint name="rear_caster_joint" type="continuous">
     <parent link="base_link"/>
     <child link="rear_caster"/>
     <origin xyz="-0.25 0 0.04" rpy="0 0 0"/>
+    <axis xyz="0 1 0"/>
+  </joint>
+  <link name="left_stabilizer">
+    <collision>
+      <origin xyz="0 0 0" rpy="0 0 0"/>
+      <geometry><sphere radius="0.04"/></geometry>
+    </collision>
+    <xacro:sphere_inertia m="1.0" r="0.04"/>
+  </link>
+  <joint name="left_stabilizer_joint" type="continuous">
+    <parent link="base_link"/>
+    <child link="left_stabilizer"/>
+    <origin xyz="0 0.25 0.04" rpy="0 0 0"/>
+    <axis xyz="0 1 0"/>
+  </joint>
+  <link name="right_stabilizer">
+    <collision>
+      <origin xyz="0 0 0" rpy="0 0 0"/>
+      <geometry><sphere radius="0.04"/></geometry>
+    </collision>
+    <xacro:sphere_inertia m="1.0" r="0.04"/>
+  </link>
+  <joint name="right_stabilizer_joint" type="continuous">
+    <parent link="base_link"/>
+    <child link="right_stabilizer"/>
+    <origin xyz="0 -0.25 0.04" rpy="0 0 0"/>
+    <axis xyz="0 1 0"/>
   </joint>
   <joint name="base_joint" type="fixed">
@@ -53,4 +91,10 @@
     <mu1>0.0</mu1><mu2>0.0</mu2>
   </gazebo>
+  <gazebo reference="left_stabilizer">
+    <mu1>0.0</mu1><mu2>0.0</mu2>
+  </gazebo>
+  <gazebo reference="right_stabilizer">
+    <mu1>0.0</mu1><mu2>0.0</mu2>
+  </gazebo>
   <gazebo reference="left_wheel">
     <mu1>1000.0</mu1><mu2>1000.0</mu2>
@@ -65,9 +109,9 @@
       <origin xyz="0 0 0" rpy="${mesh_rpy}"/>
       <geometry>
-        <mesh filename="package://archer_description/meshes/torso.obj" scale="1.0 1.0 1.0"/>
+        <mesh filename="file://$(find archer_description)/meshes/torso.obj" scale="1.0 1.0 1.0"/>
       </geometry>
     </visual>
     <collision><geometry><box size="0.2 0.3 0.15"/></geometry></collision>
-    <xacro:ballast_inertia m="5.0" w="0.2" h="0.3" d="0.15"/>
+    <xacro:box_inertia m="5.0" w="0.2" h="0.3" d="0.15"/>
   </link>
   <!-- Wheels (Hidden visually inside/under the signature Neo white sneakers) -->
@@ -104,5 +148,5 @@
       <origin xyz="0 0 0" rpy="${mesh_rpy}"/>
       <geometry>
-        <mesh filename="package://archer_description/meshes/abdomen.obj" scale="1.0 1.0 1.0"/>
+        <mesh filename="file://$(find archer_description)/meshes/abdomen.obj" scale="1.0 1.0 1.0"/>
       </geometry>
     </visual>
@@ -120,5 +164,5 @@
       <origin xyz="0 0 0.1" rpy="${mesh_rpy}"/>
       <geometry>
-        <mesh filename="package://archer_description/meshes/scapula.obj" scale="1.0 1.0 1.0"/>
+        <mesh filename="file://$(find archer_description)/meshes/scapula.obj" scale="1.0 1.0 1.0"/>
       </geometry>
     </visual>
@@ -136,5 +180,5 @@
       <origin xyz="0 0 0" rpy="${mesh_rpy}"/>
       <geometry>
-        <mesh filename="package://archer_description/meshes/head.obj" scale="1.0 1.0 1.0"/>
+        <mesh filename="file://$(find archer_description)/meshes/head.obj" scale="1.0 1.0 1.0"/>
       </geometry>
     </visual>
@@ -153,4 +197,17 @@
     <origin xyz="0.2 0 0.1" rpy="0 0 0"/>
   </joint>
+  <!-- Stereo Camera Links (cuVSLAM) — 12 cm baseline, child of head_camera_link -->
+  <link name="camera_left_link"/>
+  <joint name="camera_left_joint" type="fixed">
+    <parent link="head_camera_link"/>
+    <child link="camera_left_link"/>
+    <origin xyz="0 0.06 0" rpy="0 0 0"/>
+  </joint>
+  <link name="camera_right_link"/>
+  <joint name="camera_right_joint" type="fixed">
+    <parent link="head_camera_link"/>
+    <child link="camera_right_link"/>
+    <origin xyz="0 -0.06 0" rpy="0 0 0"/>
+  </joint>
   <link name="base_lidar_link"/>
   <joint name="base_lidar_joint" type="fixed">
@@ -172,5 +229,5 @@
         <origin xyz="0 0 0" rpy="${mesh_rpy}"/>
         <geometry>
-          <mesh filename="package://archer_description/meshes/thigh.obj" scale="1.0 1.0 1.0"/>
+          <mesh filename="file://$(find archer_description)/meshes/thigh.obj" scale="1.0 1.0 1.0"/>
         </geometry>
       </visual>
@@ -187,5 +244,5 @@
         <origin xyz="0 0 0" rpy="${mesh_rpy}"/>
         <geometry>
-          <mesh filename="package://archer_description/meshes/shin.obj" scale="1.0 1.0 1.0"/>
+          <mesh filename="file://$(find archer_description)/meshes/shin.obj" scale="1.0 1.0 1.0"/>
         </geometry>
       </visual>
@@ -238,5 +295,5 @@
         <origin xyz="0 0 0" rpy="${mesh_rpy}"/>
         <geometry>
-          <mesh filename="package://archer_description/meshes/upper_arm.obj" scale="1.0 1.0 1.0"/>
+          <mesh filename="file://$(find archer_description)/meshes/upper_arm.obj" scale="1.0 1.0 1.0"/>
         </geometry>
       </visual>
@@ -253,5 +310,5 @@
         <origin xyz="0 0 0" rpy="${mesh_rpy}"/>
         <geometry>
-          <mesh filename="package://archer_description/meshes/forearm.obj" scale="1.0 1.0 1.0"/>
+          <mesh filename="file://$(find archer_description)/meshes/forearm.obj" scale="1.0 1.0 1.0"/>
         </geometry>
       </visual>
@@ -269,5 +326,5 @@
         <origin xyz="0 0 0" rpy="1.5707963 3.14159265 1.5707963"/>
         <geometry>
-          <mesh filename="package://archer_description/meshes/palm.obj" scale="1.0 1.0 1.0"/>
+          <mesh filename="file://$(find archer_description)/meshes/palm.obj" scale="1.0 1.0 1.0"/>
         </geometry>
       </visual>

File: ros2_ws/src/archer_description/urdf/archer_gazebo.xacro (robot description, xacro)
@@ -4,7 +4,11 @@
     <!-- Joint State Publisher (Fixes No Transform error) -->
     <plugin filename="gz-sim-joint-state-publisher-system" name="gz::sim::systems::JointStatePublisher">
-      <topic>joint_states</topic>
+      <topic>/joint_states</topic>
       <joint_name>left_wheel_joint</joint_name>
       <joint_name>right_wheel_joint</joint_name>
+      <joint_name>front_caster_joint</joint_name>
+      <joint_name>rear_caster_joint</joint_name>
+      <joint_name>left_stabilizer_joint</joint_name>
+      <joint_name>right_stabilizer_joint</joint_name>
     </plugin>
     <plugin filename="gz-sim-diff-drive-system" name="gz::sim::systems::DiffDrive">
@@ -20,16 +24,17 @@
       <odom_topic>/odom</odom_topic>
       <tf_topic>/tf</tf_topic>
+      <publish_odom>true</publish_odom>
       <publish_odom_tf>true</publish_odom_tf>
       <frame_id>odom</frame_id>
-      <child_frame_id>base_link</child_frame_id>
+      <child_frame_id>base_footprint</child_frame_id>
     </plugin>
   </gazebo>
   <!-- Sensors Definition -->
   <gazebo reference="head_camera_link">
-    <!-- RGB Camera (Proven to work on WSL) -->
+    <!-- RGB Monocular Camera (for YOLO — kept on original topic) -->
     <sensor name="head_camera" type="camera">
       <pose>0 0 0 0 0 0</pose>
       <always_on>1</always_on>
-      <update_rate>2</update_rate>
+      <update_rate>30</update_rate>
       <visualize>true</visualize>
       <topic>/archer/camera/image_raw</topic>
@@ -39,6 +44,6 @@
         <horizontal_fov>1.047</horizontal_fov>
         <image>
-          <width>320</width>
-          <height>240</height>
+          <width>640</width>
+          <height>480</height>
           <format>R8G8B8</format>
         </image>
@@ -46,9 +51,9 @@
       </camera>
     </sensor>
-    <!-- Depth Camera for 3D Voxels -->
+    <!-- Depth Camera (for OctoMap / depth_to_pointcloud) -->
     <sensor name="head_camera_depth" type="depth_camera">
       <pose>0 0 0 0 0 0</pose>
       <always_on>1</always_on>
-      <update_rate>5</update_rate>
+      <update_rate>15</update_rate>
       <visualize>false</visualize>
       <topic>/archer/camera/depth</topic>
@@ -58,8 +63,50 @@
         <horizontal_fov>1.047</horizontal_fov>
         <image>
-          <width>320</width>
-          <height>240</height>
+          <width>640</width>
+          <height>480</height>
         </image>
         <clip><near>0.1</near><far>10.0</far></clip>
+      </camera>
+    </sensor>
+  </gazebo>
+  <!-- Stereo Left Camera (cuVSLAM) -->
+  <gazebo reference="camera_left_link">
+    <sensor name="camera_left" type="camera">
+      <pose>0 0 0 0 0 0</pose>
+      <always_on>1</always_on>
+      <update_rate>30</update_rate>
+      <visualize>false</visualize>
+      <topic>/archer/camera/left/image_raw</topic>
+      <gz_frame_id>camera_left_link</gz_frame_id>
+      <frame_id>camera_left_link</frame_id>
+      <camera>
+        <horizontal_fov>1.047</horizontal_fov>
+        <image>
+          <width>640</width>
+          <height>480</height>
+          <format>R8G8B8</format>
+        </image>
+        <clip><near>0.1</near><far>100</far></clip>
+      </camera>
+    </sensor>
+  </gazebo>
+  <!-- Stereo Right Camera (cuVSLAM) -->
+  <gazebo reference="camera_right_link">
+    <sensor name="camera_right" type="camera">
+      <pose>0 0 0 0 0 0</pose>
+      <always_on>1</always_on>
+      <update_rate>30</update_rate>
+      <visualize>false</visualize>
+      <topic>/archer/camera/right/image_raw</topic>
+      <gz_frame_id>camera_right_link</gz_frame_id>
+      <frame_id>camera_right_link</frame_id>
+      <camera>
+        <horizontal_fov>1.047</horizontal_fov>
+        <image>
+          <width>640</width>
+          <height>480</height>
+          <format>R8G8B8</format>
+        </image>
+        <clip><near>0.1</near><far>100</far></clip>
       </camera>
     </sensor>
@@ -86,5 +133,5 @@
         </scan>
         <range>
-          <min>0.40</min>
+          <min>0.60</min>
           <max>12.0</max>
           <resolution>0.01</resolution>
